File: Hardware/CH32V003.kicad_sch (KiCad schematic)
At the start: 10 parts, among them J7 Program, SW1 SW_SPST, U5 CH32V003F4U6, X1 X322525MOB4SI

Commit message: added photo
Parts:
- J7: footprint Connector_PinHeader_2.54mm:PinHeader_1x03_P2.54mm_Vertical -> Connector_JST:JST_XH_B3B-XH-A_1x03_P2.50mm_Vertical
Changed lines of the file:
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@@
 			)
 		)
-		(property "Footprint" "Connector_PinHeader_2.54mm:PinHeader_1x03_P2.54mm_Vertical"
+		(property "Footprint" "Connector_JST:JST_XH_B3B-XH-A_1x03_P2.50mm_Vertical"
 			(at 69.85 142.24 0)
 			(hide yes)
