File: Hardware/MMS3_hat_HC-SR04-HX711.kicad_pcb (KiCad board)
At the start: 2 copper layers, 100 x 50 mm, 63 parts, among them J1 Chainbus in, J10 Conn_01x04_Pin, J11 Conn_01x04_Pin, J2 Chainbus Out, J3 Conn_01x04_Pin, J4 Debug_USART_TX, J5 Conn_01x04_Pin, J6 Conn_01x04_Pin, J7 Program, J8 Conn_01x04_Pin, J9 Conn_01x04_Pin, Q3 MMBT3906, U1 SN74CB3Q3245PWR, U2 M24C64, U3 AMS1117, U5 CH32V003F4U6, U6 HX711_C6705483

Commit message: added photo
Parts:
- removed H7, H8, H9: ~, PCM_JLCPCB:Hole_Tooling_JLCPCB
- J7: footprint Connector_PinHeader_2.54mm:PinHeader_1x03_P2.54mm_Vertical -> Connector_JST:JST_XH_B3B-XH-A_1x03_P2.50mm_Vertical
- moved J7 0.15 mm to (136.2, 107.7), turned to 180 degrees
Connections:
- J1 pad 25: unconnected-(J1-Pin_25-Pad25) -> /Interboard_connector/R1
- J1 pad 27: unconnected-(J1-Pin_27-Pad27) -> /Interboard_connector/R2
- J2 pad 25: unconnected-(J2-Pin_25-Pad25) -> /Interboard_connector/R1
- J2 pad 27: unconnected-(J2-Pin_27-Pad27) -> /Interboard_connector/R2
Routing:
- net /Interboard_connector/R2: track 0.00 -> 4.30 mm, vias 0 -> 1
- net /Interboard_connector/R1: track 0.00 -> 4.00 mm, vias 0 -> 1
Other:
- board text added: "Hat HC-SR04 HX711 Version 1.1 Made by Wojciech Szafrański"
- board text removed: "Version 1.1 Made by Wojciech Szafrański"
