File: Hardware/MMS3_hat_HC-SR04-HX711.kicad_sch (KiCad schematic)
At the start: 14 parts, among them J4 Debug_USART_TX, U3 AMS1117

Commit message: added photo
Parts:
- removed H7, H8, H9: (no value), PCM_JLCPCB:Hole_Tooling_JLCPCB, symbol PCM_JLCPCB-Manufacturing:Tooling Hole, PCM_JLCPCB, 1.152mm
